File: design/seeed-xiao-esp32s3-expander.kicad_pcb (KiCad board)
At the start: 2 copper layers, 17.8 x 21.4 mm, 12 parts, among them J1 Conn_01x07, J2 Conn_01x07, J3 30pin, J4 Conn_01x02, J5 Conn_01x01

Commit message: Replace GPIO21 breakout with 3V3
Parts:
- renumbered GPIO21 to +3V3
Connections:
- +3V3 pad : GPIO21 -> +3V3
- J1 pad 7: GPIO21 -> +3V3
Routing:
- net GPIO21: vias 1 -> 0
- net +3V3: vias 1 -> 2
Changed lines of the file:
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@@
 		(sheetname "/")
 		(sheetfile "seeed-xiao-esp32s3-expander.kicad_sch")
+		(units
+			(unit
+				(name "A")
+				(pins "1")
+			)
+		)
 		(attr through_hole)
 		(duplicate_pad_numbers_are_jumpers no)
@@
 		(descr "Wire Pad, Square, SMD Pad,  2mm x 4mm")
 		(tags "MeasurementPoint Square SMDPad 2mmx4mm ")
-		(property "Reference" "GPIO21"
+		(property "Reference" "+3V3"
 			(at 0 2.35 0)
 			(layer "F.SilkS")
@@
 			(size 1.7 0.8)
 			(layers "F.Cu" "F.Mask")
-			(net "GPIO21")
+			(net "+3V3")
 		)
 		(pad "" smd roundrect
@@
 			(layers "F.Cu" "F.Mask")
 			(roundrect_rratio 0.25)
-			(net "GPIO21")
+			(net "+3V3")
 		)
 		(embedded_fonts no)
@@
 			(layers "*.Cu" "*.Mask")
 			(remove_unused_layers no)
-			(net "GPIO21")
+			(net "+3V3")
 			(pinfunction "Pin_7_7")
 			(pintype "passive")
@@
 		(net "GPIO18")
 	)
-	(via
-		(at 122.02 126)
-		(size 1.5)
-		(drill 1)
-		(layers "F.Cu" "B.Cu")
-		(locked yes)
-		(net "GPIO21")
-	)
 	(segment
 		(start 119.360598 127.139402)
@@
 		(net "+3V3")
 	)
+	(via
+		(at 122.02 126)
+		(size 1.5)
+		(drill 1)
+		(layers "F.Cu" "B.Cu")
+		(locked yes)
+		(net "+3V3")
+	)

Commit message: Finish routing gpio
Routing:
- net GPIO47: track 0.00 -> 10.7 mm, vias 0 -> 1
- net VIN: track 2.91 -> 13.4 mm, vias 0 -> 1
- net GPIO14: track 0.00 -> 10.5 mm
- net GPIO16: track 0.00 -> 10.2 mm
- net GPIO15: track 0.00 -> 9.33 mm
- net GPIO48: track 0.51 -> 9.18 mm, vias 0 -> 1
- net GPIO17: track 0.00 -> 7.63 mm
- net GPIO18: track 0.00 -> 6.23 mm
- net +3V3: track 1.62 -> 5.08 mm
- net unconnected-(J3-Pad10): track 2.61 -> 0.00 mm
- net unconnected-(J3-Pad8): track 2.17 -> 0.00 mm
- net unconnected-(J3-Pad6): track 1.68 -> 0.00 mm
- net unconnected-(J3-Pad13): track 1.58 -> 0.00 mm
- net GPIO21: track 1.15 -> 0.00 mm
- net GND: track 3.34 -> 4.38 mm, vias 11 -> 8
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Other:
- board size 17.8 x 21.4 mm -> 17.8 x 14 mm

Commit message: Fill ground planes
Routing:
- net unconnected-(J3-Pad11): track 1.67 -> 0.00 mm
- net unconnected-(J3-Pad9): track 1.18 -> 0.00 mm
- net GND: track 4.38 -> 4.76 mm, vias 8 -> 6
Other:
- board text added: "XIAO ESP32-S3 GPIO Expander"
- board text added: "[lg]"
- board text added: "v1"
- board text removed: "3V3"
- board text removed: "BUSY"
- board text removed: "D5"
- board text removed: "D6"
- board text removed: "D7"
- board text removed: "DIO1"
- board text removed: "MISO"
- board text removed: "MOSI"
- board text removed: "NSS"
- board text removed: "RF-SW"
- board text removed: "RST"
- board text removed: "SCK"
- board text removed: "Wio-SX1262 for XIAO V1.1"
